Commit message: update: base_link to camera_link

File: zed_wrapper/urdf/zed_descr.urdf.xacro (robot description, xacro)
@@ -18,5 +18,5 @@
   <xacro:arg name="camera_name"   default="zed" />
   <xacro:arg name="camera_model"  default="zed" />
-  <xacro:arg name="base_frame"    default="base_link" />
+  <xacro:arg name="base_frame"    default="camera_link" />
   <xacro:arg name="cam_pos_x"     default="0.0" />
   <xacro:arg name="cam_pos_y"     default="0.0" />

File: zed_wrapper/urdf/zed_macro.urdf.xacro (robot description, xacro)
@@ -55,8 +55,8 @@
     </xacro:if>
     <!-- Camera mounting point (the threaded screw hole in the bottom) -->
-    <link name="${name}_base_link" />
+    <link name="${name}_camera_link" />
     <joint name="${name}_base_joint" type="fixed">
       <parent link="${parent}"/>
-      <child link="${name}_base_link"/>
+      <child link="${name}_camera_link"/>
       <xacro:insert_block name="origin" />
     </joint>
@@ -77,5 +77,5 @@
     </link>
     <joint name="${name}_camera_center_joint" type="fixed">
-      <parent link="${name}_base_link"/>
+      <parent link="${name}_camera_link"/>
       <child link="${name}_camera_center"/>
       <origin xyz="0 0 ${height/2}" rpy="0 ${bottom_slope} 0" />
